File: vcu.brd (EAGLE design)
At the start: 34 x 40 mm, 26 parts, among them IC1 7812DT, IC2 MCP2551/SN, U1 ATMEGA328P-AU

Commit message: routing
Routing:
- net GND: track 0.00 -> 137.3 mm, vias 0 -> 4
- net +5V: track 0.00 -> 103.5 mm, vias 0 -> 6
- net N$39: track 0.00 -> 90.5 mm, vias 0 -> 1
- net B5/SCK: track 0.00 -> 77.0 mm, vias 0 -> 2
- net C3/CRX: track 0.00 -> 76.9 mm, vias 0 -> 2
- net RESET: track 0.00 -> 54.3 mm, vias 0 -> 3
- net N$40: track 0.00 -> 49.9 mm
- net C2/CTX: track 0.00 -> 46.8 mm, vias 0 -> 2
- net B4/MISO: track 0.00 -> 32.2 mm
- net N$2: track 0.00 -> 30.8 mm
- net C5: track 0.00 -> 29.1 mm
- net B3/MOSI: track 0.00 -> 25.4 mm
- net AREF: track 0.00 -> 25.1 mm
- net C4: track 0.00 -> 25.0 mm
- net N$8: track 0.00 -> 22.4 mm, vias 0 -> 3
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- added copper zone on layer 1, net GND
- added copper zone on layer 16, net GND

Commit message: provisional board
Routing:
- net +5V: track 103.5 -> 102.5 mm
- net C3/CRX: track 76.9 -> 77.5 mm
Other:
- board text added: "+5V"
- board text added: "100"
- board text added: "100nf"
- board text added: "10k"
- board text added: "120"
- board text added: "220"
- board text added: "330nf"
- board text added: "4.7K"
- board text added: "560pf"
- board text added: "ADC6"
- board text added: "ADC7"
- board text added: "AMPERSAND VCU"
- board text added: "AREF"
- board text added: "B0"
- board text added: "B1"
- board text added: "B2"
- board text added: "B3"
- board text added: "B4"
- board text added: "B5"
- board text added: "B6"
- board text added: "B7"
- board text added: "C0"
- board text added: "C1"
- board text added: "C2/CTX"
- board text added: "C3/CRX"
- board text added: "C4"
- board text added: "C5"
- board text added: "CAN H"
- board text added: "CAN L"
- board text added: "D0"
- board text added: "D1"
- board text added: "D2"
- board text added: "D3"
- board text added: "D4"
- board text added: "D5"
- board text added: "D6"
- board text added: "D7"
- board text added: "GND"
- board text added: "Green"
- board text added: "Red"
- board text added: "Rev 1.0"
- board text added: "VCC"

Commit message: semi-final
Other:
- board size 34 x 40 mm -> 33 x 40 mm
Changed lines of the file:
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@@
 <drawing>
 <settings>
-<setting alwaysvectorfont="no"/>
+<setting alwaysvectorfont="yes"/>
 <setting verticaltext="up"/>
 </settings>
-<grid distance="1" unitdist="mm" unit="mm" style="lines" multiple="1" display="yes" altdistance="5" altunitdist="mil" altunit="mil"/>
+<grid distance="0.2" unitdist="mm" unit="mm" style="lines" multiple="1" display="yes" altdistance="5" altunitdist="mil" altunit="mil"/>
 <layers>
 <layer number="1" name="Top" color="4" fill="1" visible="yes" active="yes"/>
@@
 <layer number="43" name="vRestrict" color="2" fill="10" visible="no" active="yes"/>
 <layer number="44" name="Drills" color="7" fill="1" visible="no" active="yes"/>
-<layer number="45" name="Holes" color="7" fill="1" visible="no" active="yes"/>
+<layer number="45" name="Holes" color="7" fill="1" visible="yes" active="yes"/>
 <layer number="46" name="Milling" color="3" fill="1" visible="no" active="yes"/>
 <layer number="47" name="Measures" color="7" fill="1" visible="no" active="yes"/>
@@
 <board>
 <plain>
-<wire x1="19" y1="31" x2="53" y2="31" width="0" layer="20"/>
-<wire x1="53" y1="31" x2="53" y2="71" width="0" layer="20"/>
-<wire x1="53" y1="71" x2="19" y2="71" width="0" layer="20"/>
+<wire x1="19" y1="31" x2="52" y2="31" width="0" layer="20"/>
+<wire x1="52" y1="31" x2="52" y2="71" width="0" layer="20"/>
+<wire x1="52" y1="71" x2="19" y2="71" width="0" layer="20"/>
 <wire x1="19" y1="71" x2="19" y2="31" width="0" layer="20"/>
 <text x="24.6" y="31.6" size="0.8128" layer="25">B0</text>
@@
 <text x="45.4" y="41.6" size="0.6096" layer="25">ADC6</text>
 <text x="45.4" y="39.2" size="0.6096" layer="25">ADC7</text>
-<text x="46.2" y="36.6" size="0.6096" layer="25">+5V</text>
+<text x="45.8" y="36.6" size="0.6096" layer="25">+5V</text>
 <text x="46.6" y="56.9" size="0.6096" layer="25">C0</text>
 <text x="46.7" y="54.2" size="0.6096" layer="25">C1</text>
@@
 <text x="21.2" y="61.2" size="0.6096" layer="25">GND</text>
 <hole x="20.8" y="69.2" drill="3"/>
-<hole x="51.2" y="69.2" drill="3"/>
-<hole x="51.2" y="32.8" drill="3"/>
+<hole x="50.2" y="69.2" drill="3"/>
+<hole x="50.2" y="32.8" drill="3"/>
 <hole x="20.8" y="32.8" drill="3"/>
 <text x="35" y="46" size="0.6096" layer="25">AMPERSAND VCU</text>
@@
 <polygon width="0.254" layer="1">
 <vertex x="19" y="71"/>
-<vertex x="53" y="71"/>
-<vertex x="53" y="31"/>
+<vertex x="52" y="71"/>
+<vertex x="52" y="31"/>
 <vertex x="19" y="31"/>
 </polygon>
 <polygon width="0.254" layer="16">
 <vertex x="19" y="71"/>
-<vertex x="53" y="71"/>
-<vertex x="53" y="31"/>
+<vertex x="52" y="71"/>
+<vertex x="52" y="31"/>
 <vertex x="19" y="31"/>
 </polygon>
@@
 <wire x1="49.3776" y1="43.1292" x2="48.6156" y2="43.1292" width="0.1524" layer="1"/>
 <wire x1="50.1396" y1="42.3672" x2="49.3776" y2="43.1292" width="0.1524" layer="1"/>
-<wire x1="50.1396" y1="36.2712" x2="50.1396" y2="42.3672" width="0.1524" layer="1"/>
-<wire x1="48.1584" y1="34.29" x2="50.1396" y2="36.2712" width="0.1524" layer="1"/>
-<wire x1="45.72" y1="34.29" x2="48.1584" y2="34.29" width="0.1524" layer="1"/>
+<wire x1="50.1396" y1="36.8712" x2="50.1396" y2="42.3672" width="0.1524" layer="1"/>
+<wire x1="47.5584" y1="34.29" x2="50.1396" y2="36.8712" width="0.1524" layer="1"/>
+<wire x1="45.72" y1="34.29" x2="47.5584" y2="34.29" width="0.1524" layer="1"/>
 </signal>
 <signal name="B0">
